Commit message: Update camera frames to comply with convetion

File: robotiq_hande_description/urdf/robotiq_hande.urdf.xacro (robot description, xacro)
@@ -150,4 +150,5 @@
   <link name="camera_link">
     <visual>
+    <origin xyz="0 0 0" rpy="0 ${pi/2} 0"/>
       <geometry>
         <mesh filename="package://closed_loop_dalsa_description/meshes/realsense_D405.stl"/>
@@ -156,4 +157,5 @@
     </visual>
     <collision>
+    <origin xyz="0 0 0" rpy="0 ${pi/2} 0"/>
       <geometry>
         <mesh filename="package://closed_loop_dalsa_description/meshes/realsense_D405.stl"/>
@@ -168,5 +170,5 @@
     <parent link="camera_mount"/>
     <child link="camera_link"/>
-    <origin xyz="0.01 0 0.023" rpy="0 ${95*pi/180} 0"/>
+    <origin xyz="0.01 0 0.023" rpy="0 ${5*pi/180} 0"/>
   </joint>
   <link name="camera_link_optical"/>
@@ -174,7 +176,7 @@
     <parent link="camera_link"/>
     <child link="camera_link_optical"/>
-    <origin xyz="0 0 0" rpy=" 0 ${-pi/2} 0"/>
+    <origin xyz="0 0 0" rpy="${-pi/2} 0 ${-pi/2}"/>
   </joint>
-  <gazebo reference="camera_link_optical">
+  <gazebo reference="camera_link">
     <sensor name="wrist_camera" type="rgbd_camera">
         <camera>
@@ -185,5 +187,5 @@
           </image>
           <clip><near>0.1</near><far>10</far></clip>
-          <optical_frame_id>camera_link_optical</optical_frame_id>
+          <optical_frame_id>camera_link</optical_frame_id>
         </camera>
         <always_on>1</always_on>

Commit message: New fingers

File: robotiq_hande_description/urdf/robotiq_hande.urdf.xacro (robot description, xacro)
@@ -73,19 +73,19 @@
     <parent link="gripper_body"/>
     <child link="tcp_link"/>
-    <origin xyz="0 0 0.13" rpy="0 0 0"/>
+    <origin xyz="-0.0071 0 0.174" rpy="0 ${pi/4} ${pi}"/>
   </joint>
   <!-- Fingers -->
   <link name="finger1">
     <visual>
-      <origin xyz="0 0 0" rpy="0 0 0"/>
+      <origin xyz="0 -0.025 0" rpy="0 0 0"/>
       <geometry>
-        <mesh filename="package://robotiq_hande_description/meshes/finger1_v2.stl"/>
+        <mesh filename="package://robotiq_hande_description/meshes/finger-full-v3-right.stl"/>
       </geometry>
       <material name="gray"><color rgba="0.4 0.4 0.4 1.0"/></material>
     </visual>
     <collision>
-      <origin xyz="0.01 -0.076 0.04" rpy="0 0 0"/>
+      <origin xyz="0.005 -0.078 0.09" rpy="0 ${-pi/4} 0"/>
       <geometry>
-        <box size="0.02 0.002 0.06" />
+        <box size="0.01 0.002 0.02" />
       </geometry>
     </collision>
@@ -103,14 +103,14 @@
    <link name="finger2">
     <visual>
-      <origin xyz="0 0 0" rpy="0 0 0"/>
+      <origin xyz="0 0.025 0" rpy="0 0 0"/>
       <geometry>
-        <mesh filename="package://robotiq_hande_description/meshes/finger1_v2.stl"/>
+        <mesh filename="package://robotiq_hande_description/meshes/finger-full-v3-left.stl"/>
       </geometry>
       <material name="gray"><color rgba="0.4 0.4 0.4 1.0"/></material>
     </visual>
     <collision>
-      <origin xyz="0.01 -0.076 0.04" rpy="0 0 0"/>
+      <origin xyz="-0.02 0.078 0.09" rpy="0 ${-pi/4} 0"/>
       <geometry>
-        <box size="0.02 0.002 0.06" />
+        <box size="0.01 0.002 0.02" />
       </geometry>
     </collision>
@@ -123,7 +123,7 @@
      <parent link="gripper_body"/>
      <child link="finger2"/>
-     <origin xyz="0.01443 -0.011 0.0839" rpy="0 0 ${pi}"/>
-     <axis xyz="0 1 0"/><limit lower="-0.003" upper="0.025" effort="500" velocity="0.1" acceleration="0.1"/>
-     <mimic joint="finger_joint" multiplier="1.0" offset="0.0"/>
+     <origin xyz="0.01443 -0.011 0.0839" rpy="0 0 0"/>
+     <axis xyz="0 1 0"/><limit lower="-0.025" upper="0.003" effort="500" velocity="0.1" acceleration="0.1"/>
+     <mimic joint="finger_joint" multiplier="-1.0" offset="0.0"/>
   </joint>
   <!-- Camera mount -->
