Commit message: feat: integrate Realsense D405 camera with Gazebo sensor support and bridge configuration

File: robotiq_hande_description/urdf/robotiq_hande.urdf.xacro (robot description, xacro)
@@ -98,4 +98,83 @@
       <mimic joint="finger_joint" multiplier="1.0" offset="0.0"/>
     </joint>
+    <!-- Camera Mount -->
+    <link name="camera_mount">
+      <visual>
+        <origin xyz="0 0 0" rpy="0 0 0"/>
+        <geometry>
+          <mesh filename="package://robotiq_hande_description/meshes/camera_mount_95.stl"/>
+        </geometry>
+        <material name="black"><color rgba="0.1 0.1 0.1 1.0"/></material>
+      </visual>
+      <collision>
+        <origin xyz="0 0 0" rpy="0 0 0"/>
+        <geometry>
+          <mesh filename="package://robotiq_hande_description/meshes/camera_mount_95.stl"/>
+        </geometry>
+      </collision>
+      <inertial>
+        <mass value="0.05"/>
+        <origin xyz="0 0 0" rpy="0 0 0"/>
+        <inertia ixx="0.00005" ixy="0" ixz="0" iyy="0.00005" iyz="0" izz="0.00005"/>
+      </inertial>
+    </link>
+    <joint name="camera_mount_joint" type="fixed">
+      <parent link="gripper_body"/>
+      <child link="camera_mount"/>
+      <origin xyz="-0.031 0 0.0898" rpy="0 ${-pi/2} 0"/>
+    </joint>
+    <!-- Camera -->
+    <link name="camera_link">
+      <visual>
+        <origin xyz="0 0 0" rpy="0 ${pi/2} 0"/>
+        <geometry>
+          <mesh filename="package://robotiq_hande_description/meshes/realsense_D405.stl"/>
+        </geometry>
+        <material name="black"><color rgba="0.1 0.1 0.1 1.0"/></material>
+      </visual>
+      <collision>
+        <origin xyz="0 0 0" rpy="0 ${pi/2} 0"/>
+        <geometry>
+          <mesh filename="package://robotiq_hande_description/meshes/realsense_D405.stl"/>
+        </geometry>
+      </collision>
+      <inertial>
+        <mass value="0.072"/>
+        <origin xyz="0 0 0" rpy="0 0 0"/>
+        <inertia ixx="0.00005" ixy="0" ixz="0" iyy="0.00005" iyz="0" izz="0.00005"/>
+      </inertial>
+    </link>
+    <joint name="camera_joint" type="fixed">
+      <parent link="camera_mount"/>
+      <child link="camera_link"/>
+      <origin xyz="0.01 0 0.023" rpy="0 ${5*pi/180} 0"/>
+    </joint>
+    <link name="camera_link_optical"/>
+    <joint name="camera_optical_joint" type="fixed">
+      <parent link="camera_link"/>
+      <child link="camera_link_optical"/>
+      <origin xyz="0 0 0" rpy="${-pi/2} 0 ${-pi/2}"/>
+    </joint>
+    <!-- Gazebo sensor definition -->
+    <gazebo reference="camera_link">
+      <sensor name="wrist_camera" type="rgbd_camera">
+        <camera>
+          <horizontal_fov>1.047</horizontal_fov>
+          <image>
+            <width>320</width>
+            <height>240</height>
+          </image>
+          <clip>
+            <near>0.1</near>
+            <far>10</far>
+          </clip>
+          <optical_frame_id>camera_link</optical_frame_id>
+        </camera>
+        <always_on>1</always_on>
+        <update_rate>10</update_rate>
+        <visualize>true</visualize>
+        <topic>wrist_camera</topic>
+      </sensor>
+    </gazebo>
     <!-- Gazebo ROS2 Control definition (only when sim_gazebo is true) -->
     <xacro:if value="${sim_gazebo}">

Commit message: Upgrade gripper controller to JointTrajectoryController and add new finger mesh files

File: robotiq_hande_description/urdf/robotiq_hande.urdf.xacro (robot description, xacro)
@@ -97,4 +97,56 @@
       <limit lower="0.0" upper="0.025" effort="130" velocity="0.15"/>
       <mimic joint="finger_joint" multiplier="1.0" offset="0.0"/>
+    </joint>
+    <!-- Top Finger (attached to Left Fingerbase) -->
+    <link name="top_finger">
+      <visual>
+        <origin xyz="0 0 0" rpy="0 0 0"/>
+        <geometry>
+          <mesh filename="package://robotiq_hande_description/meshes/top-finger-v1.stl"/>
+        </geometry>
+        <material name="gray"><color rgba="0.4 0.4 0.4 1.0"/></material>
+      </visual>
+      <collision>
+        <origin xyz="0 0 0" rpy="0 0 0"/>
+        <geometry>
+          <mesh filename="package://robotiq_hande_description/meshes/top-finger-v1.stl"/>
+        </geometry>
+      </collision>
+      <inertial>
+        <mass value="0.03"/>
+        <origin xyz="0.006 -0.021 0.037" rpy="0 0 0"/>
+        <inertia ixx="0.00001" ixy="0" ixz="0" iyy="0.00001" iyz="0" izz="0.00001"/>
+      </inertial>
+    </link>
+    <joint name="top_finger_joint" type="fixed">
+      <parent link="left_fingerbase"/>
+      <child link="top_finger"/>
+      <origin xyz="0 0 0" rpy="0 0 0"/>
+    </joint>
+    <!-- Bottom Finger (attached to Right Fingerbase) -->
+    <link name="bottom_finger">
+      <visual>
+        <origin xyz="0 0 0" rpy="0 0 0"/>
+        <geometry>
+          <mesh filename="package://robotiq_hande_description/meshes/bottom-finger-v1.stl"/>
+        </geometry>
+        <material name="gray"><color rgba="0.4 0.4 0.4 1.0"/></material>
+      </visual>
+      <collision>
+        <origin xyz="0 0 0" rpy="0 0 0"/>
+        <geometry>
+          <mesh filename="package://robotiq_hande_description/meshes/bottom-finger-v1.stl"/>
+        </geometry>
+      </collision>
+      <inertial>
+        <mass value="0.03"/>
+        <origin xyz="-0.022 0.021 0.037" rpy="0 0 0"/>
+        <inertia ixx="0.00001" ixy="0" ixz="0" iyy="0.00001" iyz="0" izz="0.00001"/>
+      </inertial>
+    </link>
+    <joint name="bottom_finger_joint" type="fixed">
+      <parent link="right_fingerbase"/>
+      <child link="bottom_finger"/>
+      <origin xyz="0 0 0" rpy="0 0 0"/>
     </joint>
     <!-- Camera Mount -->

Commit message: Update TCP

File: robotiq_hande_description/urdf/robotiq_hande.urdf.xacro (robot description, xacro)
@@ -39,5 +39,5 @@
       <parent link="gripper_body"/>
       <child link="tcp_link"/>
-      <origin xyz="0 0 0.100" rpy="0 0 0"/>
+      <origin xyz="-0.0264 0 0.178" rpy="0 ${-3*pi/4} 0"/>
     </joint>
     <!-- Left Fingerbase -->
