Commit message: Update tcp orientation

File: robotiq_hande_description/urdf/finger_aluminum.xacro (robot description, xacro)
@@ -12,5 +12,5 @@
       <parent link="${tcp_parent}"/>
       <child link="tcp_link"/>
-      <origin xyz="0 0 0.15" rpy="0 0 0"/>
+      <origin xyz="0 0 0.15" rpy="0 ${pi} 0"/>
     </joint>
     <!-- Top Finger (attached to Left Fingerbase) -->
