Commit message: Added realsense driver

File: robotiq_hande_description/urdf/robotiq_hande_macro.xacro (robot description, xacro)
@@ -167,4 +167,11 @@
       <origin xyz="0 0 0" rpy="${-pi/2} 0 ${-pi/2}"/>
     </joint>
+    <!-- RealSense driver root frame alias -->
+    <link name="wrist_camera_link"/>
+    <joint name="wrist_camera_joint" type="fixed">
+      <parent link="camera_link"/>
+      <child link="wrist_camera_link"/>
+      <origin xyz="0 0 0" rpy="0 0 0"/>
+    </joint>
   </xacro:macro>
 </robot>
