Commit message: Updated Hand-E body and fingerbases

File: robotiq_hande_description/urdf/gripper.urdf.xacro (robot description, xacro)
@@ -1,16 +1,13 @@
 <?xml version="1.0"?>
-<robot xmlns:xacro="http://wiki.ros.org/xacro" name="bio_lab">
-  <!-- <xacro:include filename="$(find ur_description)/urdf/ur_macro.xacro"/>
-  <xacro:include filename="$(find ur_simulation_gz)/urdf/ur_gz.ros2_control.xacro" /> -->
+<robot xmlns:xacro="http://wiki.ros.org/xacro" name="robotiq_hande">
   <xacro:include filename="$(find robotiq_hande_description)/urdf/robotiq_hande.urdf.xacro" />
   <link name="world"/>
-  <xacro:robotiq_hande_gripper parent="world">
+  <xacro:robotiq_hande_gripper parent="world" sim_gazebo="true">
     <origin xyz="0 0 0" rpy="0 0 0"/>
   </xacro:robotiq_hande_gripper>
-  <!-- <gazebo>
+  <gazebo>
     <plugin filename="gz_ros2_control-system" name="gz_ros2_control::GazeboSimROS2ControlPlugin">
-      <parameters>$(find ur_simulation_gz)/config/ur_controllers.yaml</parameters>
-      <parameters>$(find robotiq_hande_moveit_config)/config/ros2_controllers.yaml</parameters>
+      <parameters>$(find robotiq_hande_control)/config/controllers.yaml</parameters>
     </plugin>
-  </gazebo> -->
-  </robot>
+  </gazebo>
+</robot>

File: robotiq_hande_description/urdf/robotiq_hande.urdf.xacro (robot description, xacro)
@@ -1,197 +1,120 @@
 <?xml version="1.0"?>
 <robot xmlns:xacro="http://www.ros.org/wiki/xacro" name="robotiq_hande">
-  <xacro:macro name="robotiq_hande_gripper" params="parent *origin">
-    <!-- Adapter (base of the gripper) -->
-    <joint name="adapter_joint" type="fixed">
-       <xacro:insert_block name="origin" />
-       <parent link="${parent}"/>
-       <child link="gripper_adapter"/>
+  <xacro:macro name="robotiq_hande_gripper" params="parent *origin sim_gazebo:=false">
+    <!-- Gripper Base Joint connecting parent to gripper_body -->
+    <joint name="gripper_base_joint" type="fixed">
+      <xacro:insert_block name="origin" />
+      <parent link="${parent}"/>
+      <child link="gripper_body"/>
     </joint>
-    <link name="gripper_adapter">
+    <!-- Gripper Body -->
+    <link name="gripper_body">
       <visual>
         <origin xyz="0 0 0" rpy="0 0 0"/>
         <geometry>
-          <mesh filename="package://robotiq_hande_description/meshes/robotiq_adapter.stl"/>
+          <mesh filename="package://robotiq_hande_description/meshes/hand-e-body.stl"/>
+        </geometry>
+        <material name="gray"><color rgba="0.4 0.4 0.4 1.0"/></material>
+      </visual>
+      <collision>
+        <origin xyz="0 0 0" rpy="0 0 0"/>
+        <geometry>
+          <mesh filename="package://robotiq_hande_description/meshes/hand-e-body.stl"/>
+        </geometry>
+      </collision>
+      <inertial>
+        <mass value="0.86"/>
+        <origin xyz="0 0 0.042" rpy="0 0 0"/>
+        <inertia ixx="0.001" ixy="0" ixz="0" iyy="0.001" iyz="0" izz="0.001"/>
+      </inertial>
+    </link>
+    <!-- Tool Center Point (TCP) -->
+    <link name="tcp_link">
+      <inertial>
+        <mass value="0.001"/>
+        <inertia ixx="0.00001" ixy="0" ixz="0" iyy="0.00001" iyz="0" izz="0.00001"/>
+      </inertial>
+    </link>
+    <joint name="tcp_joint" type="fixed">
+      <parent link="gripper_body"/>
+      <child link="tcp_link"/>
+      <origin xyz="0 0 0.100" rpy="0 0 0"/>
+    </joint>
+    <!-- Left Fingerbase -->
+    <link name="left_fingerbase">
+      <visual>
+        <origin xyz="0 0 0" rpy="0 0 0"/>
+        <geometry>
+          <mesh filename="package://robotiq_hande_description/meshes/left_fingerbase.stl"/>
         </geometry>
         <material name="black"><color rgba="0.1 0.1 0.1 1.0"/></material>
       </visual>
       <collision>
+        <origin xyz="0 0 0" rpy="0 0 0"/>
         <geometry>
-          <mesh filename="package://robotiq_hande_description/meshes/robotiq_adapter.stl"/>
+          <mesh filename="package://robotiq_hande_description/meshes/left_fingerbase.stl"/>
         </geometry>
       </collision>
       <inertial>
-        <mass value="0.1"/>
-        <inertia ixx="0.0001" ixy="0" ixz="0" iyy="0.0001" iyz="0" izz="0.0001"/>
+        <mass value="0.05"/>
+        <origin xyz="0 0.008 -0.008" rpy="0 0 0"/>
+        <inertia ixx="0.00001" ixy="0" ixz="0" iyy="0.00001" iyz="0" izz="0.00001"/>
       </inertial>
     </link>
-    <ros2_control name="GripperHardware" type="system">
-      <hardware>
-        <plugin>gz_ros2_control/GazeboSimSystem</plugin>
-      </hardware>
-      <joint name="finger_joint">
-        <command_interface name="position" />
-        <state_interface name="position" />
-        <state_interface name="velocity" />
-        <state_interface name="effort"/>
-      </joint>
-      <joint name="finger2_joint">
-        <state_interface name="position" />
-        <state_interface name="velocity" />
-        <state_interface name="effort"/>
-      </joint>
-    </ros2_control>
+    <joint name="finger_joint" type="prismatic">
+      <parent link="gripper_body"/>
+      <child link="left_fingerbase"/>
+      <origin xyz="-0.01425 -0.022014 0.11430" rpy="0 0 0"/>
+      <axis xyz="0 1 0"/>
+      <limit lower="0.0" upper="0.025" effort="130" velocity="0.15"/>
+    </joint>
+    <!-- Right Fingerbase -->
+    <link name="right_fingerbase">
+      <visual>
+        <origin xyz="0 0 0" rpy="0 0 0"/>
+        <geometry>
+          <mesh filename="package://robotiq_hande_description/meshes/right_fingerbase.stl"/>
+        </geometry>
+        <material name="black"><color rgba="0.1 0.1 0.1 1.0"/></material>
+      </visual>
+      <collision>
+        <origin xyz="0 0 0" rpy="0 0 0"/>
+        <geometry>
+          <mesh filename="package://robotiq_hande_description/meshes/right_fingerbase.stl"/>
+        </geometry>
+      </collision>
+      <inertial>
+        <mass value="0.05"/>
+        <origin xyz="0 -0.008 -0.008" rpy="0 0 0"/>
+        <inertia ixx="0.00001" ixy="0" ixz="0" iyy="0.00001" iyz="0" izz="0.00001"/>
+      </inertial>
+    </link>
+    <joint name="finger2_joint" type="prismatic">
+      <parent link="gripper_body"/>
+      <child link="right_fingerbase"/>
+      <origin xyz="0.01425 0.022014 0.11430" rpy="0 0 0"/>
+      <axis xyz="0 -1 0"/>
+      <limit lower="0.0" upper="0.025" effort="130" velocity="0.15"/>
+      <mimic joint="finger_joint" multiplier="1.0" offset="0.0"/>
+    </joint>
+    <!-- Gazebo ROS2 Control definition (only when sim_gazebo is true) -->
+    <xacro:if value="${sim_gazebo}">
+      <ros2_control name="GripperHardware" type="system">
+        <hardware>
+          <plugin>gz_ros2_control/GazeboSimSystem</plugin>
+        </hardware>
+        <joint name="finger_joint">
+          <command_interface name="position" />
+          <state_interface name="position" />
+          <state_interface name="velocity" />
+          <state_interface name="effort"/>
+        </joint>
+        <joint name="finger2_joint">
+          <state_interface name="position" />
+          <state_interface name="velocity" />
+          <state_interface name="effort"/>
+        </joint>
+      </ros2_control>
+    </xacro:if>
   </xacro:macro>
-  <!-- Gripper body -->
-  <link name="gripper_body">
-    <visual>
-      <origin xyz="0 0 0" rpy="0 0 0"/>
-      <geometry>
-        <mesh filename="package://robotiq_hande_description/meshes/Gripper_body.stl"/>
-      </geometry>
-      <material name="gray"><color rgba="0.4 0.4 0.4 1.0"/></material>
-    </visual>
-    <collision>
-      <geometry>
-        <mesh filename="package://robotiq_hande_description/meshes/Gripper_body.stl"/>
-      </geometry>
-    </collision>
-  </link>
-  <joint name="gripper_body_joint" type="fixed">
-     <parent link="gripper_adapter"/>
-     <child link="gripper_body"/>
-     <origin xyz="0 0 0.01" rpy="0 0 0"/>
-   </joint>
-  <!-- Tool Center Point (TCP) -->
-  <link name="tcp_link">
-    <inertial>
-      <mass value="0.01"/>
-      <inertia ixx="0.00001" ixy="0" ixz="0" iyy="0.00001" iyz="0" izz="0.00001"/>
-    </inertial>
-  </link>
-  <joint name="tcp_joint" type="fixed">
-    <parent link="gripper_body"/>
-    <child link="tcp_link"/>
-    <origin xyz="-0.0071 0 0.174" rpy="0 ${pi/4} ${pi}"/>
-  </joint>
-  <!-- Fingers -->
-  <link name="finger1">
-    <visual>
-      <origin xyz="0 -0.025 0" rpy="0 0 0"/>
-      <geometry>
-        <mesh filename="package://robotiq_hande_description/meshes/finger-full-v3-right.stl"/>
-      </geometry>
-      <material name="gray"><color rgba="0.4 0.4 0.4 1.0"/></material>
-    </visual>
-    <collision>
-      <origin xyz="0.005 -0.078 0.09" rpy="0 ${-pi/4} 0"/>
-      <geometry>
-        <box size="0.01 0.002 0.02" />
-      </geometry>
-    </collision>
-    <inertial>
-      <mass value="0.1"/>
-      <inertia ixx="0.0001" ixy="0" ixz="0" iyy="0.0001" iyz="0" izz="0.0001"/>
-    </inertial>
-  </link>
-  <joint name="finger_joint" type="prismatic">
-     <parent link="gripper_body"/>
-     <child link="finger1"/>
-     <origin xyz="-0.01443 0.011 0.0839" rpy="0 0 0"/>
-     <axis xyz="0 1 0"/><limit lower="-0.003" upper="0.025" effort="500" velocity="0.1" acceleration="0.1"/>
-   </joint>
-   <link name="finger2">
-    <visual>
-      <origin xyz="0 0.025 0" rpy="0 0 0"/>
-      <geometry>
-        <mesh filename="package://robotiq_hande_description/meshes/finger-full-v3-left.stl"/>
-      </geometry>
-      <material name="gray"><color rgba="0.4 0.4 0.4 1.0"/></material>
-    </visual>
-    <collision>
-      <origin xyz="-0.02 0.078 0.09" rpy="0 ${-pi/4} 0"/>
-      <geometry>
-        <box size="0.01 0.002 0.02" />
-      </geometry>
-    </collision>
-    <inertial>
-      <mass value="0.1"/>
-      <inertia ixx="0.0001" ixy="0" ixz="0" iyy="0.0001" iyz="0" izz="0.0001"/>
-    </inertial>
-  </link>
-  <joint name="finger2_joint" type="prismatic">
-     <parent link="gripper_body"/>
-     <child link="finger2"/>
-     <origin xyz="0.01443 -0.011 0.0839" rpy="0 0 0"/>
-     <axis xyz="0 1 0"/><limit lower="-0.025" upper="0.003" effort="500" velocity="0.1" acceleration="0.1"/>
-     <mimic joint="finger_joint" multiplier="-1.0" offset="0.0"/>
-  </joint>
-  <!-- Camera mount -->
-  <link name="camera_mount">
-    <visual>
-      <origin xyz="0 0 0" rpy="0 0 0"/>
-      <geometry>
-        <mesh filename="package://closed_loop_dalsa_description/meshes/camera_mount_95.stl"/>
-      </geometry>
-      <material name="black"><color rgba="0.1 0.1 0.1 1.0"/></material>
-    </visual>
-    <collision>
-      <geometry>
-        <mesh filename="package://closed_loop_dalsa_description/meshes/camera_mount_95.stl"/>
-      </geometry>
-    </collision>
-  </link>
-  <joint name="camera_mount_joint" type="fixed">
-     <parent link="gripper_body"/>
-     <child link="camera_mount"/>
-     <origin xyz="-0.031 0 0.0755" rpy="0 ${-pi/2} 0"/>
-   </joint>
-  <!-- Camera -->
-  <link name="camera_link">
-    <visual>
-    <origin xyz="0 0 0" rpy="0 ${pi/2} 0"/>
-      <geometry>
-        <mesh filename="package://closed_loop_dalsa_description/meshes/realsense_D405.stl"/>
-      </geometry>
-      <material name="black"><color rgba="0.1 0.1 0.1 1.0"/></material>
-    </visual>
-    <collision>
-    <origin xyz="0 0 0" rpy="0 ${pi/2} 0"/>
-      <geometry>
-        <mesh filename="package://closed_loop_dalsa_description/meshes/realsense_D405.stl"/>
-      </geometry>
-    </collision>
-    <inertial>
-      <mass value="0.1"/>
-      <inertia ixx="0.0001" ixy="0" ixz="0" iyy="0.0001" iyz="0" izz="0.0001"/>
-    </inertial>
-  </link>
-  <joint name="camera_joint" type="fixed">
-    <parent link="camera_mount"/>
-    <child link="camera_link"/>
-    <origin xyz="0.01 0 0.023" rpy="0 ${5*pi/180} 0"/>
-  </joint>
-  <link name="camera_link_optical"/>
-  <joint name="camera_optical_joint" type="fixed">
-    <parent link="camera_link"/>
-    <child link="camera_link_optical"/>
-    <origin xyz="0 0 0" rpy="${-pi/2} 0 ${-pi/2}"/>
-  </joint>
-  <gazebo reference="camera_link">
-    <sensor name="wrist_camera" type="rgbd_camera">
-        <camera>
-          <horizontal_fov>1.047</horizontal_fov>
-          <image>
-            <width>320</width>
-            <height>240</height>
-          </image>
-          <clip><near>0.1</near><far>10</far></clip>
-          <optical_frame_id>camera_link</optical_frame_id>
-        </camera>
-        <always_on>1</always_on>
-        <update_rate>10</update_rate>
-        <visualize>true</visualize>
-        <topic>wrist_camera</topic>
-    </sensor>
-  </gazebo>
 </robot>

File: robotiq_hande_moveit_config/config/robotiq_hande.ros2_control.xacro (robot description, xacro)
@@ -15,4 +15,10 @@
                 <state_interface name="velocity"/>
             </joint>
+            <joint name="finger2_joint">
+                <param name="mimic">finger_joint</param>
+                <param name="multiplier">1</param>
+                <state_interface name="position"/>
+                <state_interface name="velocity"/>
+            </joint>
         </ros2_control>
     </xacro:macro>

File: robotiq_hande_moveit_config/config/robotiq_hande.urdf.xacro (robot description, xacro)
@@ -6,4 +6,8 @@
     <!-- Import control_xacro -->
     <xacro:include filename="robotiq_hande.ros2_control.xacro" />
+    <link name="world"/>
+    <xacro:robotiq_hande_gripper parent="world" sim_gazebo="false">
+        <origin xyz="0 0 0" rpy="0 0 0"/>
+    </xacro:robotiq_hande_gripper>
     <xacro:robotiq_hande_ros2_control name="FakeSystem" initial_positions_file="$(arg initial_positions_file)"/>
 </robot>

Commit message: Refactor the code and added simple aluminium fingers

File: robotiq_hande_description/urdf/gripper.urdf.xacro (robot description, xacro)
@@ -1,9 +1,14 @@
 <?xml version="1.0"?>
 <robot xmlns:xacro="http://wiki.ros.org/xacro" name="robotiq_hande">
-  <xacro:include filename="$(find robotiq_hande_description)/urdf/robotiq_hande.urdf.xacro" />
+  <!-- Include the split macros -->
+  <xacro:include filename="$(find robotiq_hande_description)/urdf/robotiq_hande_macro.xacro" />
+  <xacro:include filename="$(find robotiq_hande_description)/urdf/robotiq_hande.ros2_control.xacro" />
   <link name="world"/>
-  <xacro:robotiq_hande_gripper parent="world" sim_gazebo="true">
+  <!-- 1. Physical Geometry (Removed the old sim_gazebo flag) -->
+  <xacro:robotiq_hande_gripper parent="world">
     <origin xyz="0 0 0" rpy="0 0 0"/>
   </xacro:robotiq_hande_gripper>
+  <!-- 2. Control and Sensors (Passing sim_gz for Jazzy) -->
+  <xacro:robotiq_hande_ros2_control sim_gz="true" />
   <gazebo>
     <plugin filename="gz_ros2_control-system" name="gz_ros2_control::GazeboSimROS2ControlPlugin">

File: robotiq_hande_description/urdf/robotiq_hande.urdf.xacro (robot description, xacro)
@@ -17,8 +17,14 @@
         <material name="gray"><color rgba="0.4 0.4 0.4 1.0"/></material>
       </visual>
-      <collision>
+      <!-- <collision>
         <origin xyz="0 0 0" rpy="0 0 0"/>
         <geometry>
           <mesh filename="package://robotiq_hande_description/meshes/hand-e-body.stl"/>
+        </geometry>
+      </collision> -->
+      <collision>
+        <origin xyz="0 0 ${0.099/2}" rpy="0 0 0"/>
+        <geometry>
+          <cylinder length="0.099" radius="${0.0375 + 0.001}"/>
         </geometry>
       </collision>
@@ -103,5 +109,5 @@
         <origin xyz="0 0 0" rpy="0 0 0"/>
         <geometry>
-          <mesh filename="package://robotiq_hande_description/meshes/top-finger-v1.stl"/>
+          <mesh filename="package://robotiq_hande_description/meshes/alum-finger.stl"/>
         </geometry>
         <material name="gray"><color rgba="0.4 0.4 0.4 1.0"/></material>
@@ -110,5 +116,5 @@
         <origin xyz="0 0 0" rpy="0 0 0"/>
         <geometry>
-          <mesh filename="package://robotiq_hande_description/meshes/top-finger-v1.stl"/>
+          <mesh filename="package://robotiq_hande_description/meshes/alum-finger.stl"/>
         </geometry>
       </collision>
@@ -122,5 +128,5 @@
       <parent link="left_fingerbase"/>
       <child link="top_finger"/>
-      <origin xyz="0 0 0" rpy="0 0 0"/>
+      <origin xyz="0 0 0" rpy="0 0 ${-pi/2}"/>
     </joint>
     <!-- Bottom Finger (attached to Right Fingerbase) -->
@@ -129,5 +135,5 @@
         <origin xyz="0 0 0" rpy="0 0 0"/>
         <geometry>
-          <mesh filename="package://robotiq_hande_description/meshes/bottom-finger-v1.stl"/>
+          <mesh filename="package://robotiq_hande_description/meshes/alum-finger.stl"/>
         </geometry>
         <material name="gray"><color rgba="0.4 0.4 0.4 1.0"/></material>
@@ -136,5 +142,5 @@
         <origin xyz="0 0 0" rpy="0 0 0"/>
         <geometry>
-          <mesh filename="package://robotiq_hande_description/meshes/bottom-finger-v1.stl"/>
+          <mesh filename="package://robotiq_hande_description/meshes/alum-finger.stl"/>
         </geometry>
       </collision>
@@ -148,5 +154,5 @@
       <parent link="right_fingerbase"/>
       <child link="bottom_finger"/>
-      <origin xyz="0 0 0" rpy="0 0 0"/>
+      <origin xyz="0 0 0" rpy="0 0 ${pi/2}"/>
     </joint>
     <!-- Camera Mount -->

File: robotiq_hande_moveit_config/config/robotiq_hande.urdf.xacro (robot description, xacro)
@@ -3,5 +3,5 @@
     <xacro:arg name="initial_positions_file" default="initial_positions.yaml" />
     <!-- Import robotiq_hande urdf file -->
-    <xacro:include filename="$(find robotiq_hande_description)/urdf/robotiq_hande.urdf.xacro" />
+    <xacro:include filename="$(find robotiq_hande_description)/urdf/robotiq_hande_macro.xacro" />
     <!-- Import control_xacro -->
     <xacro:include filename="robotiq_hande.ros2_control.xacro" />

Commit message: Added parameter to choose fingers

File: robotiq_hande_description/urdf/gripper.urdf.xacro (robot description, xacro)
@@ -5,6 +5,8 @@
   <xacro:include filename="$(find robotiq_hande_description)/urdf/robotiq_hande.ros2_control.xacro" />
   <link name="world"/>
+  <!-- Finger configuration parameter -->
+  <xacro:arg name="finger_type" default="aluminum" />
   <!-- 1. Physical Geometry (Removed the old sim_gazebo flag) -->
-  <xacro:robotiq_hande_gripper parent="world">
+  <xacro:robotiq_hande_gripper parent="world" finger_type="$(arg finger_type)">
     <origin xyz="0 0 0" rpy="0 0 0"/>
   </xacro:robotiq_hande_gripper>

File: robotiq_hande_description/urdf/robotiq_hande_macro.xacro (robot description, xacro)
@@ -1,5 +1,8 @@
 <?xml version="1.0"?>
 <robot xmlns:xacro="http://www.ros.org/wiki/xacro" name="robotiq_hande">
-  <xacro:macro name="robotiq_hande_gripper" params="parent *origin sim_gazebo:=false">
+  <!-- Include finger macros -->
+  <xacro:include filename="$(find robotiq_hande_description)/urdf/finger_aluminum.xacro" />
+  <xacro:include filename="$(find robotiq_hande_description)/urdf/finger_v1.xacro" />
+  <xacro:macro name="robotiq_hande_gripper" params="parent *origin sim_gazebo:=false finger_type:=aluminum">
     <!-- Gripper Base Joint connecting parent to gripper_body -->
     <joint name="gripper_base_joint" type="fixed">
@@ -35,25 +38,4 @@
       </inertial>
     </link>
-    <!-- Tool Center Point (TCP) -->
-    <link name="tcp_link">
-      <inertial>
-        <mass value="0.001"/>
-        <inertia ixx="0.00001" ixy="0" ixz="0" iyy="0.00001" iyz="0" izz="0.00001"/>
-      </inertial>
-      <!-- <collision>
-        <origin xyz="0 0 0" rpy="0 0 0"/>
-        <geometry>
-          <sphere radius="0.001"/>
-        </geometry>
-      </collision> -->
-    </link>
-    <joint name="tcp_joint" type="fixed">
-      <parent link="gripper_body"/>
-      <child link="tcp_link"/>
-      <origin xyz="0 0 0.15" rpy="0 0 0"/>
-    </joint>
-    <!-- <gazebo reference="tcp_joint">
-      <preserveFixedJoint>true</preserveFixedJoint>
-    </gazebo> -->
     <!-- Left Fingerbase -->
     <link name="left_fingerbase">
@@ -120,56 +102,11 @@
       </plugin>
     </gazebo> -->
-    <!-- Top Finger (attached to Left Fingerbase) -->
-    <link name="top_finger">
-      <visual>
-        <origin xyz="0 0 0" rpy="0 0 0"/>
-        <geometry>
-          <mesh filename="package://robotiq_hande_description/meshes/alum-finger.stl"/>
-        </geometry>
-        <material name="gray"><color rgba="0.4 0.4 0.4 1.0"/></material>
-      </visual>
-      <collision>
-        <origin xyz="0 0 0" rpy="0 0 0"/>
-        <geometry>
-          <mesh filename="package://robotiq_hande_description/meshes/alum-finger.stl"/>
-        </geometry>
-      </collision>
-      <inertial>
-        <mass value="0.03"/>
-        <origin xyz="0.006 -0.021 0.037" rpy="0 0 0"/>
-        <inertia ixx="0.00001" ixy="0" ixz="0" iyy="0.00001" iyz="0" izz="0.00001"/>
-      </inertial>
-    </link>
-    <joint name="top_finger_joint" type="fixed">
-      <parent link="left_fingerbase"/>
-      <child link="top_finger"/>
-      <origin xyz="0 0 0" rpy="0 0 ${-pi/2}"/>
-    </joint>
-    <!-- Bottom Finger (attached to Right Fingerbase) -->
-    <link name="bottom_finger">
-      <visual>
-        <origin xyz="0 0 0" rpy="0 0 0"/>
-        <geometry>
-          <mesh filename="package://robotiq_hande_description/meshes/alum-finger.stl"/>
-        </geometry>
-        <material name="gray"><color rgba="0.4 0.4 0.4 1.0"/></material>
-      </visual>
-      <collision>
-        <origin xyz="0 0 0" rpy="0 0 0"/>
-        <geometry>
-          <mesh filename="package://robotiq_hande_description/meshes/alum-finger.stl"/>
-        </geometry>
-      </collision>
-      <inertial>
-        <mass value="0.03"/>
-        <origin xyz="-0.022 0.021 0.037" rpy="0 0 0"/>
-        <inertia ixx="0.00001" ixy="0" ixz="0" iyy="0.00001" iyz="0" izz="0.00001"/>
-      </inertial>
-    </link>
-    <joint name="bottom_finger_joint" type="fixed">
-      <parent link="right_fingerbase"/>
-      <child link="bottom_finger"/>
-      <origin xyz="0 0 0" rpy="0 0 ${pi/2}"/>
-    </joint>
+    <!-- Finger pair and TCP selection -->
+    <xacro:if value="${finger_type in ['aluminum', 'aluminium']}">
+      <xacro:finger_aluminum parent_left="left_fingerbase" parent_right="right_fingerbase" tcp_parent="gripper_body" />
+    </xacro:if>
+    <xacro:if value="${finger_type in ['v1', 'finger_v1', 'top_bottom_v1']}">
+      <xacro:finger_v1 parent_left="left_fingerbase" parent_right="right_fingerbase" tcp_parent="gripper_body" />
+    </xacro:if>
     <!-- Camera Mount -->
     <link name="camera_mount">
