Commit message: Added option to disable camera and gripper, plus launch file for real gripper

File: robotiq_hande_description/urdf/gripper.urdf.xacro (robot description, xacro)
@@ -5,16 +5,26 @@
   <xacro:include filename="$(find robotiq_hande_description)/urdf/robotiq_hande.ros2_control.xacro" />
   <link name="world"/>
-  <!-- Finger configuration parameter -->
+  <!-- Configuration parameters -->
   <xacro:arg name="finger_type" default="aluminum" />
-  <!-- 1. Physical Geometry (Removed the old sim_gazebo flag) -->
-  <xacro:robotiq_hande_gripper parent="world" finger_type="$(arg finger_type)">
+  <xacro:arg name="use_sim" default="true" />
+  <xacro:arg name="use_camera" default="true" />
+  <xacro:arg name="com_port" default="/tmp/ttyUR" />
+  <!-- 1. Physical Geometry -->
+  <xacro:robotiq_hande_gripper parent="world" finger_type="$(arg finger_type)" load_camera="$(arg use_camera)">
     <origin xyz="0 0 0" rpy="0 0 0"/>
   </xacro:robotiq_hande_gripper>
   <!-- 2. Control and Sensors (Passing sim_gz for Jazzy) -->
-  <xacro:robotiq_hande_ros2_control sim_gz="true" />
-  <gazebo>
-    <plugin filename="gz_ros2_control-system" name="gz_ros2_control::GazeboSimROS2ControlPlugin">
-      <parameters>$(find robotiq_hande_control)/config/controllers.yaml</parameters>
-    </plugin>
-  </gazebo>
+  <xacro:robotiq_hande_ros2_control
+    sim_gz="$(arg use_sim)"
+    use_mock_hardware="false"
+    mock_gripper="false"
+    load_camera="$(arg use_camera)"
+    com_port="$(arg com_port)"/>
+  <xacro:if value="$(arg use_sim)">
+    <gazebo>
+      <plugin filename="gz_ros2_control-system" name="gz_ros2_control::GazeboSimROS2ControlPlugin">
+        <parameters>$(find robotiq_hande_control)/config/controllers.yaml</parameters>
+      </plugin>
+    </gazebo>
+  </xacro:if>
 </robot>

File: robotiq_hande_description/urdf/robotiq_hande.ros2_control.xacro (robot description, xacro)
@@ -1,27 +1,29 @@
 <?xml version="1.0"?>
 <robot xmlns:xacro="http://www.ros.org/wiki/xacro">
-  <xacro:macro name="robotiq_hande_ros2_control" params="sim_gz:=true">
+  <xacro:macro name="robotiq_hande_ros2_control" params="sim_gz:=true use_mock_hardware:=false mock_gripper:=false com_port:=/tmp/ttyUR load_camera:=true">
     <xacro:if value="${sim_gz}">
       <!-- Gazebo Camera Sensor -->
-      <gazebo reference="camera_link">
-        <sensor name="wrist_camera" type="rgbd_camera">
-          <camera>
-            <horizontal_fov>1.518436</horizontal_fov>
-            <image>
-              <width>1280</width>
-              <height>720</height>
-            </image>
-            <clip>
-              <near>0.05</near>
-              <far>10</far>
-            </clip>
-            <optical_frame_id>camera_link</optical_frame_id>
-          </camera>
-          <always_on>1</always_on>
-          <update_rate>15</update_rate>
-          <visualize>true</visualize>
-          <topic>wrist_camera</topic>
-        </sensor>
-      </gazebo>
+      <xacro:if value="${load_camera}">
+        <gazebo reference="camera_link">
+          <sensor name="wrist_camera" type="rgbd_camera">
+            <camera>
+              <horizontal_fov>1.518436</horizontal_fov>
+              <image>
+                <width>1280</width>
+                <height>720</height>
+              </image>
+              <clip>
+                <near>0.05</near>
+                <far>10</far>
+              </clip>
+              <optical_frame_id>camera_link</optical_frame_id>
+            </camera>
+            <always_on>1</always_on>
+            <update_rate>15</update_rate>
+            <visualize>true</visualize>
+            <topic>wrist_camera</topic>
+          </sensor>
+        </gazebo>
+      </xacro:if>
       <!-- Gazebo Motor Controller -->
       <ros2_control name="GripperHardware" type="system">
@@ -43,6 +45,49 @@
     </xacro:if>
     <xacro:unless value="${sim_gz}">
-       <!-- Placeholder for the real Robotiq RS485 physical interface -->
-       <!-- We will add the real driver plugin here later -->
+      <!-- Check if either full mock hardware or gripper mock hardware is requested -->
+      <xacro:if value="${use_mock_hardware or mock_gripper}">
+        <ros2_control name="GripperHardware" type="system">
+          <hardware>
+            <plugin>mock_components/GenericSystem</plugin>
+          </hardware>
+          <joint name="finger_joint">
+            <command_interface name="position" />
+            <state_interface name="position">
+              <param name="initial_value">0.0</param>
+            </state_interface>
+            <state_interface name="velocity" />
+          </joint>
+          <joint name="finger2_joint">
+            <param name="mimic">finger_joint</param>
+            <param name="multiplier">1</param>
+            <state_interface name="position" />
+            <state_interface name="velocity" />
+          </joint>
+        </ros2_control>
+      </xacro:if>
+      <xacro:unless value="${use_mock_hardware or mock_gripper}">
+        <!-- Real Robotiq Gripper Driver Interface -->
+        <ros2_control name="GripperHardware" type="system">
+          <hardware>
+            <plugin>robotiq_driver/RobotiqGripperHardwareInterface</plugin>
+            <param name="COM_port">${com_port}</param>
+            <param name="baud_rate">115200</param>
+            <param name="slave_id">9</param>
+          </hardware>
+          <joint name="finger_joint">
+            <command_interface name="position" />
+            <state_interface name="position">
+              <param name="initial_value">0.0</param>
+            </state_interface>
+            <state_interface name="velocity" />
+          </joint>
+          <joint name="finger2_joint">
+            <param name="mimic">finger_joint</param>
+            <param name="multiplier">1</param>
+            <state_interface name="position" />
+            <state_interface name="velocity" />
+          </joint>
+        </ros2_control>
+      </xacro:unless>
     </xacro:unless>
   </xacro:macro>

File: robotiq_hande_description/urdf/robotiq_hande_macro.xacro (robot description, xacro)
@@ -4,5 +4,5 @@
   <xacro:include filename="$(find robotiq_hande_description)/urdf/finger_aluminum.xacro" />
   <xacro:include filename="$(find robotiq_hande_description)/urdf/finger_v1.xacro" />
-  <xacro:macro name="robotiq_hande_gripper" params="parent *origin sim_gazebo:=false finger_type:=aluminum">
+  <xacro:macro name="robotiq_hande_gripper" params="parent *origin sim_gazebo:=false finger_type:=aluminum load_camera:=true">
     <!-- Gripper Base Joint connecting parent to gripper_body -->
     <joint name="gripper_base_joint" type="fixed">
@@ -109,69 +109,72 @@
       <xacro:finger_v1 parent_left="left_fingerbase" parent_right="right_fingerbase" tcp_parent="gripper_body" />
     </xacro:if>
-    <!-- Camera Mount -->
-    <link name="camera_mount">
-      <visual>
+    <!-- Camera Mount and Sensor (conditionally loaded) -->
+    <xacro:if value="${load_camera}">
+      <!-- Camera Mount -->
+      <link name="camera_mount">
+        <visual>
+          <origin xyz="0 0 0" rpy="0 0 0"/>
+          <geometry>
+            <mesh filename="package://robotiq_hande_description/meshes/camera_mount_95.stl"/>
+          </geometry>
+          <material name="black"><color rgba="0.1 0.1 0.1 1.0"/></material>
+        </visual>
+        <collision>
+          <origin xyz="0 0 0" rpy="0 0 0"/>
+          <geometry>
+            <mesh filename="package://robotiq_hande_description/meshes/camera_mount_95.stl"/>
+          </geometry>
+        </collision>
+        <inertial>
+          <mass value="0.05"/>
+          <origin xyz="0 0 0" rpy="0 0 0"/>
+          <inertia ixx="0.00005" ixy="0" ixz="0" iyy="0.00005" iyz="0" izz="0.00005"/>
+        </inertial>
+      </link>
+      <joint name="camera_mount_joint" type="fixed">
+        <parent link="gripper_body"/>
+        <child link="camera_mount"/>
+        <origin xyz="-0.031 0 0.0898" rpy="0 ${-pi/2} 0"/>
+      </joint>
+      <!-- Camera -->
+      <link name="camera_link">
+        <visual>
+          <origin xyz="0 0 0" rpy="0 ${pi/2} 0"/>
+          <geometry>
+            <mesh filename="package://robotiq_hande_description/meshes/realsense_D405.stl"/>
+          </geometry>
+          <material name="black"><color rgba="0.1 0.1 0.1 1.0"/></material>
+        </visual>
+        <collision>
+          <origin xyz="0 0 0" rpy="0 ${pi/2} 0"/>
+          <geometry>
+            <mesh filename="package://robotiq_hande_description/meshes/realsense_D405.stl"/>
+          </geometry>
+        </collision>
+        <inertial>
+          <mass value="0.072"/>
+          <origin xyz="0 0 0" rpy="0 0 0"/>
+          <inertia ixx="0.00005" ixy="0" ixz="0" iyy="0.00005" iyz="0" izz="0.00005"/>
+        </inertial>
+      </link>
+      <joint name="camera_joint" type="fixed">
+        <parent link="camera_mount"/>
+        <child link="camera_link"/>
+        <origin xyz="0.01 0 0.023" rpy="0 ${5*pi/180} 0"/>
+      </joint>
+      <link name="camera_link_optical"/>
+      <joint name="camera_optical_joint" type="fixed">
+        <parent link="camera_link"/>
+        <child link="camera_link_optical"/>
+        <origin xyz="0 0 0" rpy="${-pi/2} 0 ${-pi/2}"/>
+      </joint>
+      <!-- RealSense driver root frame alias -->
+      <link name="wrist_camera_link"/>
+      <joint name="wrist_camera_joint" type="fixed">
+        <parent link="camera_link"/>
+        <child link="wrist_camera_link"/>
         <origin xyz="0 0 0" rpy="0 0 0"/>
-        <geometry>
-          <mesh filename="package://robotiq_hande_description/meshes/camera_mount_95.stl"/>
-        </geometry>
-        <material name="black"><color rgba="0.1 0.1 0.1 1.0"/></material>
-      </visual>
-      <collision>
-        <origin xyz="0 0 0" rpy="0 0 0"/>
-        <geometry>
-          <mesh filename="package://robotiq_hande_description/meshes/camera_mount_95.stl"/>
-        </geometry>
-      </collision>
-      <inertial>
-        <mass value="0.05"/>
-        <origin xyz="0 0 0" rpy="0 0 0"/>
-        <inertia ixx="0.00005" ixy="0" ixz="0" iyy="0.00005" iyz="0" izz="0.00005"/>
-      </inertial>
-    </link>
-    <joint name="camera_mount_joint" type="fixed">
-      <parent link="gripper_body"/>
-      <child link="camera_mount"/>
-      <origin xyz="-0.031 0 0.0898" rpy="0 ${-pi/2} 0"/>
-    </joint>
-    <!-- Camera -->
-    <link name="camera_link">
-      <visual>
-        <origin xyz="0 0 0" rpy="0 ${pi/2} 0"/>
-        <geometry>
-          <mesh filename="package://robotiq_hande_description/meshes/realsense_D405.stl"/>
-        </geometry>
-        <material name="black"><color rgba="0.1 0.1 0.1 1.0"/></material>
-      </visual>
-      <collision>
-        <origin xyz="0 0 0" rpy="0 ${pi/2} 0"/>
-        <geometry>
-          <mesh filename="package://robotiq_hande_description/meshes/realsense_D405.stl"/>
-        </geometry>
-      </collision>
-      <inertial>
-        <mass value="0.072"/>
-        <origin xyz="0 0 0" rpy="0 0 0"/>
-        <inertia ixx="0.00005" ixy="0" ixz="0" iyy="0.00005" iyz="0" izz="0.00005"/>
-      </inertial>
-    </link>
-    <joint name="camera_joint" type="fixed">
-      <parent link="camera_mount"/>
-      <child link="camera_link"/>
-      <origin xyz="0.01 0 0.023" rpy="0 ${5*pi/180} 0"/>
-    </joint>
-    <link name="camera_link_optical"/>
-    <joint name="camera_optical_joint" type="fixed">
-      <parent link="camera_link"/>
-      <child link="camera_link_optical"/>
-      <origin xyz="0 0 0" rpy="${-pi/2} 0 ${-pi/2}"/>
-    </joint>
-    <!-- RealSense driver root frame alias -->
-    <link name="wrist_camera_link"/>
-    <joint name="wrist_camera_joint" type="fixed">
-      <parent link="camera_link"/>
-      <child link="wrist_camera_link"/>
-      <origin xyz="0 0 0" rpy="0 0 0"/>
-    </joint>
+      </joint>
+    </xacro:if>
   </xacro:macro>
 </robot>
