Commit message: Update hardware parameters and remove mimic joint from robotiq hand-e control interface

File: robotiq_hande_description/urdf/robotiq_hande.ros2_control.xacro (robot description, xacro)
@@ -71,7 +71,9 @@
           <hardware>
             <plugin>robotiq_driver/RobotiqGripperHardwareInterface</plugin>
+            <param name="gripper_profile">hand_e</param>
+            <param name="gripper_closed_position">0.025</param>
             <param name="COM_port">${com_port}</param>
-            <param name="baud_rate">115200</param>
-            <param name="slave_id">9</param>
+            <param name="baudrate">115200</param>
+            <param name="slave_address">9</param>
           </hardware>
           <joint name="finger_joint">
@@ -82,10 +84,4 @@
             <state_interface name="velocity" />
           </joint>
-          <joint name="finger2_joint">
-            <param name="mimic">finger_joint</param>
-            <param name="multiplier">1</param>
-            <state_interface name="position" />
-            <state_interface name="velocity" />
-          </joint>
         </ros2_control>
       </xacro:unless>
